File: tomahawk/tomahawk4x6/tomahawk.kicad_pcb (KiCad board)
At the start: 2 copper layers, 79 parts, among them SW1 SW_Push, SW10 SW_Push, SW11 SW_Push, SW12 SW_Push, SW13 SW_Push, SW14 SW_Push, SW15 SW_Push, SW16 SW_Push, SW17 SW_Push, SW18 SW_Push, SW19 SW_Push, SW2 SW_Push, SW20 SW_Push, SW21 SW_Push, SW22 SW_Push, SW23 SW_Push, SW24 SW_Push, SW25 SW_Push, SW26 SW_Push, SW27 SW_Push, SW28 SW_Push, SW29 SW_Push, SW3 SW_Push, SW30 SW_Push, SW31 SW_Push, SW32 SW_Push, SW33 SW_Push, SW34 SW_Push, SW35 SW_Push, SW36 SW_Push, SW37 SW_Push, SW38 SW_Push, SW39 SW_Push, SW4 SW_Push, SW5 SW_Push, SW6 SW_Push, SW7 SW_Push, SW8 SW_Push, SW9 SW_Push, U2 nice_nano

Commit message: some more
Parts:
- removed the D28 at (109.9, 110.3)
- removed the D29 at (127.9, 114.3)
- removed the D30 at (145.8, 114.8)
- removed the D31 at (91.9, 135.3)
- removed the D32 at (109.9, 127.3)
- removed the D33 at (127.9, 131.3)
- removed the SW28 at (101.0, 104.9)
- removed the SW29 at (119.0, 108.9)
- removed the SW30 at (137.0, 110.8)
- removed the SW31 at (83.0, 129.9)
- removed the SW32 at (101.0, 121.9)
- removed the SW33 at (119.0, 125.9)
- U2: footprint Scotto MCU:Nice_Nano_V2 -> nice-nano:nice_nano
- moved D26 42.5 mm to (109.9, 110.3)
- moved SW26 42.5 mm to (101.0, 104.9)
- moved D25 38.9 mm to (91.9, 118.3)
- moved SW25 38.9 mm to (83.0, 112.9)
- moved SW27 36.2 mm to (119.0, 108.9)
- moved D27 36.2 mm to (127.9, 114.3)
- moved SW28 16.7 mm to (148.6, 116.0)
- moved D28 16.7 mm to (153.6, 125.1)
- moved D29 16.7 mm to (168.4, 138.6)
- moved D30 16.7 mm to (178.5, 155.4)
- moved D31 16.7 mm to (139.6, 139.0)
- moved D32 16.7 mm to (154.3, 152.6)
- moved D33 16.7 mm to (164.6, 169.4)
- moved SW29 16.7 mm to (165.5, 128.5)
- moved SW30 16.7 mm to (178.7, 145.0)
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- renumbered D34 to D28, D35 to D29, D36 to D30, D37 to D31, D38 to D32, D39 to D33, SW34 to SW28, SW35 to SW29, SW36 to SW30, SW37 to SW31, SW38 to SW32, SW39 to SW33
Connections:
- SW25 pad 1: COL1 -> COL3
- SW26 pad 1: COL2 -> COL4
- SW27 pad 1: COL3 -> COL5
- U2 pad 1: unconnected-(U2-TX0/P0.06-Pad1) -> COL1
- U2 pad 10: COL1 -> ROW1
- U2 pad 11: COL2 -> ROW2
- U2 pad 12: COL3 -> ROW3
- U2 pad 13: COL4 -> unconnected-(U2-NFC1/P0.09-Pad13)
- U2 pad 14: COL5 -> unconnected-(U2-NFC2/P0.10-Pad14)
- U2 pad 15: COL6 -> TROW2
- U2 pad 2: ROW1 -> unconnected-(U2-RX1/P0.08-Pad2)
- U2 pad 3: ROW2 -> unconnected-(U2-GND-Pad3)
- U2 pad 4: ROW3 -> unconnected-(U2-GND-Pad4)
- U2 pad 5: ROW4 -> COL2
- U2 pad 6: ROW5 -> COL3
- U2 pad 7: ROW6 -> COL4
- U2 pad 8: TROW2 -> COL5
- U2 pad 9: TROW1 -> COL6
